File: Pi Monitor Optoisolator/Pi Monitor Optoisolator.kicad_sch (KiCad schematic)
At the start: 11 parts, among them J1 Conn_01x07_Pin, J2 Conn_01x07_Pin, Q1 WL-OCPT_SERIES_827, Q2 WL-OCPT_SERIES_827, Q3 WL-OCPT_SERIES_827

Commit message: Minor adjustments
* Renamed LICENSE to COPYING (I wish GitHub would ask you what you wanted to name the license file)
* Added a COPYRIGHT NOTICE for the Pi Monitor Optoisolator. I did this as a seperate file, because unlike actual code files, there's not a ton of room for lots of text in a schematic or PCB drawing file.
* Update .gitignore file
Other:
- title: (none) -> Pi Monitor Optoisolator Schematic
Changed lines of the file:
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@@
 	(generator "eeschema")
 	(generator_version "9.0")
-	(paper "A4")
+	(paper "USLetter")
+	(title_block
+		(title "Pi Monitor Optoisolator Schematic")
+		(date "2025-07-18")
+		(rev "v1.0")
+		(comment 1 "See details at https://github.com/jseyfert3/mcu-on-the-go")
+		(comment 2 "Released under GPL-3.0-or-later license")
+		(comment 3 "Copyright 2025 Jonathan Seyfert")
+	)
 	(wire
 		(pts

Commit message: fix: Updated PN of optoisolator
Parts:
- Q1, Q2, Q3: value WL-OCPT_SERIES_827 -> 140827181010
Changed lines of the file:
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@@
 			)
 		)
-		(property "Value" "WL-OCPT_SERIES_827"
+		(property "Value" "140827181010"
 			(at 131.0482 54.61 0)
 			(effects
@@
 			)
 		)
-		(property "Value" "WL-OCPT_SERIES_827"
+		(property "Value" "140827181010"
 			(at 131.0482 105.41 0)
 			(effects
@@
 			)
 		)
-		(property "Value" "WL-OCPT_SERIES_827"
+		(property "Value" "140827181010"
 			(at 131.0482 80.01 0)
 			(effects
